File: kicad_smd_files/Main Board Rev1/Input_stage.sch (KiCad schematic (older format))
At the start: 57 parts, among them J4 RADIO INTERFACE, J5 MIC INPUT, J6 LINE INPUT, J7 REMOTE INPUT, J8 LINK INPUT, U2 MCP6L01U, U4 SP232E, U6 LM324N

Commit message: Smaller PCB, cheaper parts
Parts:
- removed C21, C27, C30: 1uF, Capacitor_SMD:C_0402_1005Metric, symbol Device:C_Small
- removed C24, C31: 0.1uF, Capacitor_SMD:C_0402_1005Metric, symbol Device:C_Small
- removed J5: MIC INPUT, mk312-smd-footprints:SJ13515SMTTR, symbol Connector:AudioJack3_SwitchTR
- removed R17, R20: 2.2K, Resistor_SMD:R_0603_1608Metric, symbol Device:R_US
- removed R21, R22: 100K, Resistor_SMD:R_0603_1608Metric, symbol Device:R_US
- removed R27: 20K, Resistor_SMD:R_0603_1608Metric, symbol Device:R_US
- removed R28: 1M, Resistor_SMD:R_0603_1608Metric, symbol Device:R_US
- removed R29: 4.7K, Resistor_SMD:R_0603_1608Metric, symbol Device:R_US
- removed U2: MCP6L01U, Package_TO_SOT_SMD:SOT-23-5, symbol estim_parts:MCP6L01U
- C20, C34, C35, C36, C37: Manufacturer_Name Murata -> Yageo; Manufacturer_Part_Number GCM155R71C104JA55D -> CC402KRX7R7BB104; Mouser Part Number 81-GCM155R71C104JA5D -> 603-CC402KRX7R7BB104
- C22, C23, C25, C26, C28, C29, C38, C39: Manufacturer_Name Murata -> Taiyo Yuden; Manufacturer_Part_Number GRM155R61C105MA12D -> JMK105C6105MV-F; Mouser Part Number 81-GRM155R61C105MA2D -> 963-JMK105C6105MV-F
- C32, C33: Manufacturer_Name Murata -> KEMET; Manufacturer_Part_Number GCM1555C1H102JA16J -> C0402C102K5RAC7411; Mouser Part Number 81-GCM1555C1H102JA6J -> 80-C0402C102K5R7411
- D3, D4: value 1N4148W-E3-08 -> LL4148; footprint Diode_SMD:D_SOD-123 -> mk312-smd-footprints:LL4148_SOD_80; Manufacturer_Name Vishay -> ON Semiconductor; Manufacturer_Part_Number 1N4148W-E3-08 -> LL4148; Mouser Part Number 78-1N4148W-E3-08 -> 512-LL4148
- R14, R15, R16, R19: footprint Resistor_SMD:R_0603_1608Metric -> Resistor_SMD:R_0402_1005Metric; Manufacturer_Name Panasonic -> Yageo; Manufacturer_Part_Number ERJ-PA3F1001V -> RC0402FR-071KL; Mouser Part Number 667-ERJ-PA3F1001V -> 603-RC0402FR-071KL
- R18: footprint Resistor_SMD:R_0603_1608Metric -> Resistor_SMD:R_0402_1005Metric; Manufacturer_Name Panasonic -> Yageo; Manufacturer_Part_Number ERJ-PA3F1501V -> RC0402FR-071K5L; Mouser Part Number 667-ERJ-PA3F1501V -> 603-RC0402FR-071K5L
- R23, R24: footprint Resistor_SMD:R_0603_1608Metric -> Resistor_SMD:R_0402_1005Metric; Manufacturer_Name Panasonic -> Yageo; Manufacturer_Part_Number ERJ-PA3F2002V -> RC0402FR-0720KL; Mouser Part Number 667-ERJ-PA3F2002V -> 603-RC0402FR-0720KL
- R25: footprint Resistor_SMD:R_0603_1608Metric -> Resistor_SMD:R_0402_1005Metric; Manufacturer_Name Panasonic -> Yageo; Manufacturer_Part_Number ERJ-PA3F1002V -> RC0402FR-0710KL; Mouser Part Number 667-ERJ-PA3F1002V -> 603-RC0402FR-0710KL
- R26: footprint Resistor_SMD:R_0603_1608Metric -> Resistor_SMD:R_0402_1005Metric; Manufacturer_Name Panasonic -> Yageo; Manufacturer_Part_Number ERJ-PA3F4701V -> RC0402FR-074K7L; Mouser Part Number 667-ERJ-PA3F4701V -> 603-RC0402FR-074K7L
- R30, R31, R38, R39: footprint Resistor_SMD:R_0603_1608Metric -> Resistor_SMD:R_0402_1005Metric; Manufacturer_Name Panasonic -> Yageo; Manufacturer_Part_Number ERJ-PA3F1003V -> RC0402FR-07100KL; Mouser Part Number 667-ERJ-PA3F1003V -> 603-RC0402FR-07100KL
- R32, R33: value 20K -> 2K; footprint Resistor_SMD:R_0603_1608Metric -> Resistor_SMD:R_0402_1005Metric; Manufacturer_Name Panasonic -> Yageo; Manufacturer_Part_Number ERJ-PA3F2002V -> RC0402FR-072KL; Mouser Part Number 667-ERJ-PA3F2002V -> 603-RC0402FR-072KL
- R34, R35: value 1M -> 100K; footprint Resistor_SMD:R_0603_1608Metric -> Resistor_SMD:R_0402_1005Metric; Manufacturer_Name Panasonic -> Yageo; Manufacturer_Part_Number ERJ-PA3F1004V -> RC0402FR-07100KL; Mouser Part Number 667-ERJ-PA3F1004V -> 603-RC0402FR-07100KL
- R36: value 1M -> 20K; footprint Resistor_SMD:R_0603_1608Metric -> Resistor_SMD:R_0402_1005Metric; Manufacturer_Name Panasonic -> Yageo; Manufacturer_Part_Number ERJ-PA3F1004V -> RC0402FR-0720KL; Mouser Part Number 667-ERJ-PA3F1004V -> 603-RC0402FR-0720KL
- R37: value 100K -> 2K; footprint Resistor_SMD:R_0603_1608Metric -> Resistor_SMD:R_0402_1005Metric; Manufacturer_Name Panasonic -> Yageo; Manufacturer_Part_Number ERJ-PA3F1003V -> RC0402FR-072KL; Mouser Part Number 667-ERJ-PA3F1003V -> 603-RC0402FR-072KL
- U4: value SP232E -> MAX202; footprint Package_SO:SOIC-16_3.9x9.9mm_P1.27mm -> Package_SO:TSSOP-16_4.4x5mm_P0.65mm; Manufacturer_Name MaxLinear -> Texas Instruments; Manufacturer_Part_Number SP232EEN-L/TR -> MAX202CPWR; Mouser Part Number 701-SP232EEN-L/TR -> 595-MAX202CPWR
- U6: footprint Package_SO:SOIC-14_3.9x8.7mm_P1.27mm -> Package_SO:TSSOP-14_4.4x5mm_P0.65mm; Manufacturer_Part_Number LM324DR -> LM324LVIPWR; Mouser Part Number 595-LM324DR -> 595-LM324LVIPWR
Connections:
- wire segments 207 -> 166
- no-connect marks 5 -> 3
