File: kicad_smd_files/Main Board Rev1/Panel_Circuit.sch (KiCad schematic (older format))
At the start: 31 parts, among them J12 Conn_01x24_Male, Q1 MMBT3904-7-F, Q2 MMBT3904-7-F, SW2 LEFT/DOWN, SW3 OK, SW4 RIGHT/UP, SW5 MENU, U3 CD4006B

Commit message: Smaller PCB, cheaper parts
Parts:
- C19: Manufacturer_Name Murata -> Yageo; Manufacturer_Part_Number GCM155R71C104JA55D -> CC402KRX7R7BB104; Mouser Part Number 81-GCM155R71C104JA5D -> 603-CC402KRX7R7BB104
- Q1, Q2: value MMBT3904-7-F -> MMBT3904; Manufacturer_Name Diodes Incorporated -> Nexperia; Manufacturer_Part_Number MMBT3904-7-F -> MMBT3904; Mouser Part Number 621-MMBT3904-F -> 771-MMBT3904T/R
- R10, R7, R8, R9: footprint Resistor_SMD:R_0603_1608Metric -> Resistor_SMD:R_0402_1005Metric; Manufacturer_Name Panasonic -> Yageo; Manufacturer_Part_Number ERJ-PA3F3900V -> RC0402JR-07390RL; Mouser Part Number 667-ERJ-PA3F3900V -> 603-RC0402JR-07390RL
- R11: footprint Resistor_SMD:R_0603_1608Metric -> Resistor_SMD:R_0402_1005Metric; Manufacturer_Name Panasonic -> Yageo; Manufacturer_Part_Number ERJ-PA3F47R0V -> RC0402FR-0747RL; Mouser Part Number 667-ERJ-PA3F47R0V -> 603-RC0402FR-0747RL
- R12, R13: footprint Resistor_SMD:R_0603_1608Metric -> Resistor_SMD:R_0402_1005Metric; Manufacturer_Name Panasonic -> Yageo; Manufacturer_Part_Number ERJ-PA3F1501V -> RC0402FR-071K5L; Mouser Part Number 667-ERJ-PA3F1501V -> 603-RC0402FR-071K5L
- U3: value CD4006B -> CD4066B; footprint Package_SO:SOIC-14_3.9x8.7mm_P1.27mm -> Package_SO:TSSOP-14_4.4x5mm_P0.65mm; Manufacturer_Part_Number CD4066BM96 -> CD4066BPWR; Mouser Part Number 595-CD4066BM96 -> 595-CD4066BPWR
