File: kicad_smd_files/Main Board Rev1/MK312B_MCU.sch (KiCad schematic (older format))
At the start: 12 parts, among them J11 Conn_01x24_Male, J3 Conn_02x03_Odd_Even, U1 ATmega16-16AU

Commit message: Smaller PCB, cheaper parts
Parts:
- C15, C16: Manufacturer_Name Murata -> Yageo; Manufacturer_Part_Number GCM1555C1H180FA16J -> CC402JRNPO9BN180; Mouser Part Number 81-GCM1555C1H180FA6J -> 603-CC402JRNPO9BN180
- C17, C18: Manufacturer_Name Murata -> Yageo; Manufacturer_Part_Number GCM155R71C104JA55D -> CC402KRX7R7BB104; Mouser Part Number 81-GCM155R71C104JA5D -> 603-CC402KRX7R7BB104
- R3: value 100K -> 10K; footprint Resistor_SMD:R_0603_1608Metric -> Resistor_SMD:R_0402_1005Metric; Manufacturer_Name Panasonic -> Yageo; Manufacturer_Part_Number ERJ-PA3F1003V -> RC0402FR-0710KL; Mouser Part Number 667-ERJ-PA3F1003V -> 603-RC0402FR-0710KL
- R4: value 20K -> 2K; footprint Resistor_SMD:R_0603_1608Metric -> Resistor_SMD:R_0402_1005Metric; Manufacturer_Name Panasonic -> Yageo; Manufacturer_Part_Number ERJ-PA3F2002V -> RC0402FR-072KL; Mouser Part Number 667-ERJ-PA3F2002V -> 603-RC0402FR-072KL
- R5: footprint Resistor_SMD:R_0603_1608Metric -> Resistor_SMD:R_0402_1005Metric; Manufacturer_Name Panasonic -> Yageo; Manufacturer_Part_Number ERJ-PA3F1002V -> RC0402FR-0710KL; Mouser Part Number 667-ERJ-PA3F1002V -> 603-RC0402FR-0710KL
- R6: footprint Resistor_SMD:R_0603_1608Metric -> Resistor_SMD:R_0402_1005Metric; Manufacturer_Name Panasonic -> Yageo; Manufacturer_Part_Number ERJ-PA3F3301V -> RC0402JR-133K3L; Mouser Part Number 667-ERJ-PA3F3301V -> 603-RC0402JR-133K3L
Changed lines of the file:
@@
 AR Path="/5CB40F50/5E3BF956" Ref="R3"  Part="1"
 F 0 "R3" H 5750 1459 59  0000 L BNN
-F 1 "100K" H 5750 1270 59  0000 L BNN
-F 2 "Resistor_SMD:R_0603_1608Metric" H 5900 1400 50  0001 C CNN
+F 1 "10K" H 5750 1270 59  0000 L BNN
+F 2 "Resistor_SMD:R_0402_1005Metric" H 5900 1400 50  0001 C CNN
 F 3 "https://www.mouser.com/datasheet/2/315/AOA0000C331-1141874.pdf" H 5900 1400 50  0001 C CNN
-F 4 "Panasonic" H 5900 1400 50  0001 C CNN "Manufacturer_Name"
-F 5 "ERJ-PA3F1003V" H 5900 1400 50  0001 C CNN "Manufacturer_Part_Number"
-F 6 "667-ERJ-PA3F1003V" H 5900 1400 50  0001 C CNN "Mouser Part Number"
+F 4 "Yageo" H 5900 1400 50  0001 C CNN "Manufacturer_Name"
+F 5 "RC0402FR-0710KL" H 5900 1400 50  0001 C CNN "Manufacturer_Part_Number"
+F 6 "603-RC0402FR-0710KL" H 5900 1400 50  0001 C CNN "Mouser Part Number"
 	1    5900 1400
 	1    0    0    -1
@@
 AR Path="/5CB40F50/0D06550A" Ref="R4"  Part="1"
 F 0 "R4" H 5750 2159 59  0000 L BNN
-F 1 "20K" H 5750 1970 59  0000 L BNN
-F 2 "Resistor_SMD:R_0603_1608Metric" H 5900 2100 50  0001 C CNN
+F 1 "2K" H 5750 1970 59  0000 L BNN
+F 2 "Resistor_SMD:R_0402_1005Metric" H 5900 2100 50  0001 C CNN
 F 3 "https://www.mouser.com/datasheet/2/315/AOA0000C331-1141874.pdf" H 5900 2100 50  0001 C CNN
-F 4 "Panasonic" H 5900 2100 50  0001 C CNN "Manufacturer_Name"
-F 5 "ERJ-PA3F2002V" H 5900 2100 50  0001 C CNN "Manufacturer_Part_Number"
-F 6 "667-ERJ-PA3F2002V" H 5900 2100 50  0001 C CNN "Mouser Part Number"
+F 4 "Yageo" H 5900 2100 50  0001 C CNN "Manufacturer_Name"
+F 5 "RC0402FR-072KL" H 5900 2100 50  0001 C CNN "Manufacturer_Part_Number"
+F 6 "603-RC0402FR-072KL" H 5900 2100 50  0001 C CNN "Mouser Part Number"
 	1    5900 2100
 	1    0    0    -1
@@
 F 0 "R6" H 6150 2159 59  0000 L BNN
 F 1 "3.3K" H 6150 1970 59  0000 L BNN
-F 2 "Resistor_SMD:R_0603_1608Metric" H 6300 2100 50  0001 C CNN
+F 2 "Resistor_SMD:R_0402_1005Metric" H 6300 2100 50  0001 C CNN
 F 3 "https://www.mouser.com/datasheet/2/315/AOA0000C331-1141874.pdf" H 6300 2100 50  0001 C CNN
-F 4 "Panasonic" H 6300 2100 50  0001 C CNN "Manufacturer_Name"
-F 5 "ERJ-PA3F3301V" H 6300 2100 50  0001 C CNN "Manufacturer_Part_Number"
-F 6 "667-ERJ-PA3F3301V" H 6300 2100 50  0001 C CNN "Mouser Part Number"
+F 4 "Yageo" H 6300 2100 50  0001 C CNN "Manufacturer_Name"
+F 5 "RC0402JR-133K3L" H 6300 2100 50  0001 C CNN "Manufacturer_Part_Number"
+F 6 "603-RC0402JR-133K3L" H 6300 2100 50  0001 C CNN "Mouser Part Number"
 	1    6300 2100
 	1    0    0    -1
@@
 F 0 "R5" H 6150 1459 59  0000 L BNN
 F 1 "10K" H 6150 1270 59  0000 L BNN
-F 2 "Resistor_SMD:R_0603_1608Metric" H 6300 1400 50  0001 C CNN
+F 2 "Resistor_SMD:R_0402_1005Metric" H 6300 1400 50  0001 C CNN
 F 3 "https://www.mouser.com/datasheet/2/315/AOA0000C331-1141874.pdf" H 6300 1400 50  0001 C CNN
-F 4 "Panasonic" H 6300 1400 50  0001 C CNN "Manufacturer_Name"
-F 5 "ERJ-PA3F1002V" H 6300 1400 50  0001 C CNN "Manufacturer_Part_Number"
-F 6 "667-ERJ-PA3F1002V" H 6300 1400 50  0001 C CNN "Mouser Part Number"
+F 4 "Yageo" H 6300 1400 50  0001 C CNN "Manufacturer_Name"
+F 5 "RC0402FR-0710KL" H 6300 1400 50  0001 C CNN "Manufacturer_Part_Number"
+F 6 "603-RC0402FR-0710KL" H 6300 1400 50  0001 C CNN "Mouser Part Number"
 	1    6300 1400
 	-1   0    0    1
@@
 F 2 "Capacitor_SMD:C_0402_1005Metric" H 2800 2100 50  0001 C CNN
 F 3 "https://www.mouser.com/datasheet/2/281/GCM1555C1H180FA16-01-1064431.pdf" H 2800 2100 50  0001 C CNN
-F 4 "Murata" H 2800 2100 50  0001 C CNN "Manufacturer_Name"
-F 5 "GCM1555C1H180FA16J" H 2800 2100 50  0001 C CNN "Manufacturer_Part_Number"
-F 6 "81-GCM1555C1H180FA6J" H 2800 2100 50  0001 C CNN "Mouser Part Number"
+F 4 "Yageo" H 2800 2100 50  0001 C CNN "Manufacturer_Name"
+F 5 "CC402JRNPO9BN180" H 2800 2100 50  0001 C CNN "Manufacturer_Part_Number"
+F 6 "603-CC402JRNPO9BN180" H 2800 2100 50  0001 C CNN "Mouser Part Number"
 	1    2800 2100
 	-1   0    0    -1
@@
 F 2 "Capacitor_SMD:C_0402_1005Metric" H 3200 2100 50  0001 C CNN
 F 3 "https://www.mouser.com/datasheet/2/281/GCM1555C1H180FA16-01-1064431.pdf" H 3200 2100 50  0001 C CNN
-F 4 "Murata" H 3200 2100 50  0001 C CNN "Manufacturer_Name"
-F 5 "GCM1555C1H180FA16J" H 3200 2100 50  0001 C CNN "Manufacturer_Part_Number"
-F 6 "81-GCM1555C1H180FA6J" H 3200 2100 50  0001 C CNN "Mouser Part Number"
+F 4 "Yageo" H 3200 2100 50  0001 C CNN "Manufacturer_Name"
+F 5 "CC402JRNPO9BN180" H 3200 2100 50  0001 C CNN "Manufacturer_Part_Number"
+F 6 "603-CC402JRNPO9BN180" H 3200 2100 50  0001 C CNN "Mouser Part Number"
 	1    3200 2100
 	1    0    0    -1
@@
 F 2 "Capacitor_SMD:C_0402_1005Metric" H 4200 950 50  0001 C CNN
 F 3 "https://www.mouser.com/datasheet/2/281/murata_03122018_GCM_Series-1310150.pdf" H 4200 950 50  0001 C CNN
-F 4 "Murata" H 4200 950 50  0001 C CNN "Manufacturer_Name"
-F 5 "GCM155R71C104JA55D" H 4200 950 50  0001 C CNN "Manufacturer_Part_Number"
-F 6 "81-GCM155R71C104JA5D" H 4200 950 50  0001 C CNN "Mouser Part Number"
+F 4 "Yageo" H 4200 950 50  0001 C CNN "Manufacturer_Name"
+F 5 "CC402KRX7R7BB104" H 4200 950 50  0001 C CNN "Manufacturer_Part_Number"
+F 6 "603-CC402KRX7R7BB104" H 4200 950 50  0001 C CNN "Mouser Part Number"
 	1    4200 950
 	0    1    1    0
@@
 F 2 "Capacitor_SMD:C_0402_1005Metric" H 4200 650 50  0001 C CNN
 F 3 "https://www.mouser.com/datasheet/2/281/murata_03122018_GCM_Series-1310150.pdf" H 4200 650 50  0001 C CNN
-F 4 "Murata" H 4200 650 50  0001 C CNN "Manufacturer_Name"
-F 5 "GCM155R71C104JA55D" H 4200 650 50  0001 C CNN "Manufacturer_Part_Number"
-F 6 "81-GCM155R71C104JA5D" H 4200 650 50  0001 C CNN "Mouser Part Number"
+F 4 "Yageo" H 4200 650 50  0001 C CNN "Manufacturer_Name"
+F 5 "CC402KRX7R7BB104" H 4200 650 50  0001 C CNN "Manufacturer_Part_Number"
+F 6 "603-CC402KRX7R7BB104" H 4200 650 50  0001 C CNN "Mouser Part Number"
 	1    4200 650
 	0    1    -1   0

Commit message: part footprint corrections
Parts:
- C15, C16: Manufacturer_Part_Number CC402JRNPO9BN180 -> CC0402JRNPO9BN180
Changed lines of the file:
@@
 F 3 "https://www.mouser.com/datasheet/2/281/GCM1555C1H180FA16-01-1064431.pdf" H 2800 2100 50  0001 C CNN
 F 4 "Yageo" H 2800 2100 50  0001 C CNN "Manufacturer_Name"
-F 5 "CC402JRNPO9BN180" H 2800 2100 50  0001 C CNN "Manufacturer_Part_Number"
+F 5 "CC0402JRNPO9BN180" H 2800 2100 50  0001 C CNN "Manufacturer_Part_Number"
 F 6 "603-CC402JRNPO9BN180" H 2800 2100 50  0001 C CNN "Mouser Part Number"
 	1    2800 2100
@@
 F 3 "https://www.mouser.com/datasheet/2/281/GCM1555C1H180FA16-01-1064431.pdf" H 3200 2100 50  0001 C CNN
 F 4 "Yageo" H 3200 2100 50  0001 C CNN "Manufacturer_Name"
-F 5 "CC402JRNPO9BN180" H 3200 2100 50  0001 C CNN "Manufacturer_Part_Number"
+F 5 "CC0402JRNPO9BN180" H 3200 2100 50  0001 C CNN "Manufacturer_Part_Number"
 F 6 "603-CC402JRNPO9BN180" H 3200 2100 50  0001 C CNN "Mouser Part Number"
 	1    3200 2100
