File: kicad_smd_files/Main Board Rev1/PSU.sch (KiCad schematic (older format))
At the start: 30 parts, among them IC1 LD1086BDTTR, IC2 L7805CV, IC3 L7809ABV, IC4 L7809ABV, J1 Barrel_Jack_MountingPin, J2 +12V Battery

Commit message: Smaller PCB, cheaper parts
Parts:
- added R17: 1K, Resistor_SMD:R_0402_1005Metric, symbol Device:R_US
- C1: Manufacturer_Name Panasonic -> Taiyo Yuden; Manufacturer_Part_Number EEE-FK1C100R -> TMK212BBJ106MG-T; Mouser Part Number 667-EEE-FK1C100R -> 963-TMK212BBJ106MG-T
- C10, C11, C2, C3, C6, C7, C8, C9: Manufacturer_Name Murata -> Yageo; Manufacturer_Part_Number GCM155R71C104JA55D -> CC402KRX7R7BB104; Mouser Part Number 81-GCM155R71C104JA5D -> 603-CC402KRX7R7BB104
- C13: footprint Capacitor_SMD:C_Elec_4x5.8 -> Capacitor_SMD:C_Elec_4x5.4; Manufacturer_Part_Number EEE-FK1C100R -> EEE-1CA100SR; Mouser Part Number 667-EEE-FK1C100R -> 667-EEE-1CA100SR
- C4, C5: Manufacturer_Part_Number EEE-FT1C102AP -> EEE-FK1C102SP; Mouser Part Number 667-EEE-FT1C102AP -> 667-EEE-FK1C102SP
- D1, D2: value GF1G-E3/67A -> 583-FM4004W-W; footprint mk312-smd-footprints:DO-214BA -> mk312-smd-footprints:DO-214AC; Manufacturer_Part_Number FM4004W-W -> 583-FM4004W-W
- J1: footprint Connector_BarrelJack:BarrelJack_Horizontal -> mk312-smd-footprints:DJ_Jack_PJ-003A; Manufacturer_Part_Number PJ-002A -> PJ-003A; Mouser Part Number 490-PJ-002A -> 490-PJ-003A
- R1: value 1K -> 100K; footprint Resistor_SMD:R_0603_1608Metric -> Resistor_SMD:R_0402_1005Metric; Manufacturer_Name Panasonic -> Yageo; Manufacturer_Part_Number ERJ-PA3F1001V -> RC0402FR-07100KL; Mouser Part Number 667-ERJ-PA3F1001V -> 603-RC0402FR-07100KL
- R2: value 110 -> 10K; footprint Resistor_SMD:R_0603_1608Metric -> Resistor_SMD:R_0402_1005Metric; Manufacturer_Name Panasonic -> Yageo; Manufacturer_Part_Number ERJ-PA3F1100V -> RC0402FR-0710KL; Mouser Part Number 667-ERJ-PA3F1100V -> 603-RC0402FR-0710KL
- S1: footprint mk312-smd-footprints:E-Switch_M7_SPDT -> mk312-smd-footprints:SW_E-Switch-LC-1258; Manufacturer_Part_Number 100SP1T2B4M7RE -> LC1258EENP; Mouser Part Number 612-100-A2472 -> 612-LC1258EENP
Connections:
- net at IC1.1 (ADJ), R1.1: now also R17.2; no longer R2.1
- new net: R17.1, R2.1
Other:
- moved on the sheet: R1

Commit message: part footprint corrections
Parts:
- C12, C14: footprint Capacitor_SMD:C_Elec_8x10.2 -> Capacitor_SMD:CP_Elec_8x10; Manufacturer_Name Panasonic -> Nichicon; Manufacturer_Part_Number EEE-FK1C471P -> UWT1C471MNL1GS; Mouser Part Number 667-EEE-FK1C471P -> 647-UWT1C471MNL1S
- C13: footprint Capacitor_SMD:C_Elec_4x5.4 -> Capacitor_SMD:CP_Elec_4x5.4; Manufacturer_Name Panasonic -> Nichicon; Manufacturer_Part_Number EEE-1CA100SR -> UWX1C100MCL1GB; Mouser Part Number 667-EEE-1CA100SR -> 647-UWX1C100MCL1
- C4, C5: footprint Capacitor_SMD:C_Elec_10x10.2 -> Capacitor_SMD:CP_Elec_10x10; Manufacturer_Name Panasonic -> Nichicon; Manufacturer_Part_Number EEE-FK1C102SP -> UCM1C102MNL1GS; Mouser Part Number 667-EEE-FK1C102SP -> 647-UCM1C102MNL1GS
Changed lines of the file:
@@
 F 0 "C4" H 6315 1846 50  0000 L CNN
 F 1 "1000uF" H 6315 1755 50  0000 L CNN
-F 2 "Capacitor_SMD:C_Elec_10x10.2" H 6200 1800 50  0001 C CNN
-F 3 "https://www.mouser.com/datasheet/2/315/ABA0000C1240-1130326.pdf" H 6200 1800 50  0001 C CNN
-F 4 "Panasonic" H 6200 1800 50  0001 C CNN "Manufacturer_Name"
-F 5 "EEE-FK1C102SP" H 6200 1800 50  0001 C CNN "Manufacturer_Part_Number"
-F 6 "667-EEE-FK1C102SP" H 6200 1800 50  0001 C CNN "Mouser Part Number"
+F 2 "Capacitor_SMD:CP_Elec_10x10" H 6200 1800 50  0001 C CNN
+F 3 "https://www.mouser.com/datasheet/2/293/e-ucm-883824.pdf" H 6200 1800 50  0001 C CNN
+F 4 "Nichicon" H 6200 1800 50  0001 C CNN "Manufacturer_Name"
+F 5 "UCM1C102MNL1GS" H 6200 1800 50  0001 C CNN "Manufacturer_Part_Number"
+F 6 "647-UCM1C102MNL1GS" H 6200 1800 50  0001 C CNN "Mouser Part Number"
 	1    6200 1800
 	1    0    0    -1
@@
 F 0 "C5" H 6915 1846 50  0000 L CNN
 F 1 "1000uF" H 6915 1755 50  0000 L CNN
-F 2 "Capacitor_SMD:C_Elec_10x10.2" H 6800 1800 50  0001 C CNN
-F 3 "https://www.mouser.com/datasheet/2/315/ABA0000C1240-1130326.pdf" H 6800 1800 50  0001 C CNN
-F 4 "Panasonic" H 6800 1800 50  0001 C CNN "Manufacturer_Name"
-F 5 "EEE-FK1C102SP" H 6800 1800 50  0001 C CNN "Manufacturer_Part_Number"
-F 6 "667-EEE-FK1C102SP" H 6800 1800 50  0001 C CNN "Mouser Part Number"
+F 2 "Capacitor_SMD:CP_Elec_10x10" H 6800 1800 50  0001 C CNN
+F 3 "https://www.mouser.com/datasheet/2/293/e-ucm-883824.pdf" H 6800 1800 50  0001 C CNN
+F 4 "Nichicon" H 6800 1800 50  0001 C CNN "Manufacturer_Name"
+F 5 "UCM1C102MNL1GS" H 6800 1800 50  0001 C CNN "Manufacturer_Part_Number"
+F 6 "647-UCM1C102MNL1GS" H 6800 1800 50  0001 C CNN "Mouser Part Number"
 	1    6800 1800
 	1    0    0    -1
@@
 F 0 "C13" H 11065 1796 50  0000 L CNN
 F 1 "10uF" H 11065 1705 50  0000 L CNN
-F 2 "Capacitor_SMD:C_Elec_4x5.4" H 10950 1750 50  0001 C CNN
+F 2 "Capacitor_SMD:CP_Elec_4x5.4" H 10950 1750 50  0001 C CNN
 F 3 "https://www.mouser.com/datasheet/2/315/ABA0000C1181-947564.pdf" H 10950 1750 50  0001 C CNN
-F 4 "Panasonic" H 10950 1750 50  0001 C CNN "Manufacturer_Name"
-F 5 "EEE-1CA100SR" H 10950 1750 50  0001 C CNN "Manufacturer_Part_Number"
-F 6 "667-EEE-1CA100SR" H 10950 1750 50  0001 C CNN "Mouser Part Number"
+F 4 "Nichicon" H 10950 1750 50  0001 C CNN "Manufacturer_Name"
+F 5 "UWX1C100MCL1GB" H 10950 1750 50  0001 C CNN "Manufacturer_Part_Number"
+F 6 "647-UWX1C100MCL1" H 10950 1750 50  0001 C CNN "Mouser Part Number"
 	1    10950 1750
 	1    0    0    -1
@@
 F 0 "C14" H 10965 2996 50  0000 L CNN
 F 1 "470uF" H 10965 2905 50  0000 L CNN
-F 2 "Capacitor_SMD:C_Elec_8x10.2" H 10850 2950 50  0001 C CNN
+F 2 "Capacitor_SMD:CP_Elec_8x10" H 10850 2950 50  0001 C CNN
 F 3 "https://www.mouser.com/datasheet/2/315/ABA0000C1181-947564.pdf" H 10850 2950 50  0001 C CNN
-F 4 "Panasonic" H 10850 2950 50  0001 C CNN "Manufacturer_Name"
-F 5 "EEE-FK1C471P" H 10850 2950 50  0001 C CNN "Manufacturer_Part_Number"
-F 6 "667-EEE-FK1C471P" H 10850 2950 50  0001 C CNN "Mouser Part Number"
+F 4 "Nichicon" H 10850 2950 50  0001 C CNN "Manufacturer_Name"
+F 5 "UWT1C471MNL1GS" H 10850 2950 50  0001 C CNN "Manufacturer_Part_Number"
+F 6 "647-UWT1C471MNL1S" H 10850 2950 50  0001 C CNN "Mouser Part Number"
 	1    10850 2950
 	1    0    0    -1
@@
 F 0 "C12" H 10965 4296 50  0000 L CNN
 F 1 "470uF" H 10965 4205 50  0000 L CNN
-F 2 "Capacitor_SMD:C_Elec_8x10.2" H 10850 4250 50  0001 C CNN
+F 2 "Capacitor_SMD:CP_Elec_8x10" H 10850 4250 50  0001 C CNN
 F 3 "https://www.mouser.com/datasheet/2/315/ABA0000C1181-947564.pdf" H 10850 4250 50  0001 C CNN
-F 4 "Panasonic" H 10850 4250 50  0001 C CNN "Manufacturer_Name"
-F 5 "EEE-FK1C471P" H 10850 4250 50  0001 C CNN "Manufacturer_Part_Number"
-F 6 "667-EEE-FK1C471P" H 10850 4250 50  0001 C CNN "Mouser Part Number"
+F 4 "Nichicon" H 10850 4250 50  0001 C CNN "Manufacturer_Name"
+F 5 "UWT1C471MNL1GS" H 10850 4250 50  0001 C CNN "Manufacturer_Part_Number"
+F 6 "647-UWT1C471MNL1S" H 10850 4250 50  0001 C CNN "Mouser Part Number"
 	1    10850 4250
 	1    0    0    -1
