File: kicad_smd_files/Main Board Rev1/mk312.kicad_pcb (KiCad board)
At the start: 4 copper layers, 119.6 x 88.5 mm, 158 parts, among them IC1 LD1086BDTTR, IC2 L7805CV, IC3 L7809ABV, IC4 L7809ABV, J1 Barrel_Jack_MountingPin, J10 OUTPUT B, J11 Conn_01x24_Male, J12 Conn_01x24_Male, J2 +12V Battery, J3 Conn_02x03_Odd_Even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

Commit message: Updated case design
Other:
- board text added: "MK312-BT-SMD Rev2 2019-5-27"
- board text removed: "MK312-BT-SMD Rev1 2019-5-24"
