File: kicad_smd_files/Main Board Rev1/Output_stage.sch (KiCad schematic (older format))
At the start: 41 parts, among them J10 OUTPUT B, J9 OUTPUT A, Q3 IRFR9024NTRPBF, Q4 IRLR120NTRPBF, Q5 IRFR9024NTRPBF, Q6 IRFR9024NTRPBF, Q7 IRLR120NTRPBF, Q8 IRFR9024NTRPBF, U7 LM358N, U8 LTC1661

Commit message: Some tweaks and modifications
Parts:
- Q3, Q5, Q6, Q8: value IRFR9024NTRPBF -> IRLR120NTRPBF; Manufacturer_Part_Number IRFR9024NTRPBF -> IRLR120NTRPBF; Mouser Part Number 942-IRFR9024NTRPBF -> 942-IRLR120NTRPBF
- Q4, Q7: value IRLR120NTRPBF -> IRFR9024NTRPBF; Manufacturer_Part_Number IRLR120NTRPBF -> IRFR9024NTRPBF; Mouser Part Number 942-IRLR120NTRPBF -> 942-IRFR9024NTRPBF
Changed lines of the file:
@@
 AR Path="/5CB41D9F/4F009C7F" Ref="Q3"  Part="1"
 F 0 "Q3" H 7950 1400 59  0000 L BNN
-F 1 "IRFR9024NTRPBF" H 7950 1300 59  0000 L BNN
+F 1 "IRLR120NTRPBF" H 7950 1300 59  0000 L BNN
 F 2 "Package_TO_SOT_SMD:TO-252-2" H 7700 1400 50  0001 C CNN
 F 3 "https://www.mouser.com/datasheet/2/196/irfr9024npbf-1228513.pdf" H 7700 1400 50  0001 C CNN
 F 4 "Infineon" H 7700 1400 50  0001 C CNN "Manufacturer_Name"
-F 5 "IRFR9024NTRPBF" H 7700 1400 50  0001 C CNN "Manufacturer_Part_Number"
-F 6 "942-IRFR9024NTRPBF" H 7700 1400 50  0001 C CNN "Mouser Part Number"
+F 5 "IRLR120NTRPBF" H 7700 1400 50  0001 C CNN "Manufacturer_Part_Number"
+F 6 "942-IRLR120NTRPBF" H 7700 1400 50  0001 C CNN "Mouser Part Number"
 	1    7700 1400
 	1    0    0    -1
@@
 AR Path="/5CB41D9F/91F1D459" Ref="Q5"  Part="1"
 F 0 "Q5" H 7950 3500 59  0000 L BNN
-F 1 "IRFR9024NTRPBF" H 7950 3400 59  0000 L BNN
+F 1 "IRLR120NTRPBF" H 7950 3400 59  0000 L BNN
 F 2 "Package_TO_SOT_SMD:TO-252-2" H 7700 3500 50  0001 C CNN
 F 3 "https://www.mouser.com/datasheet/2/196/irfr9024npbf-1228513.pdf" H 7700 3500 50  0001 C CNN
 F 4 "Infineon" H 7700 3500 50  0001 C CNN "Manufacturer_Name"
-F 5 "IRFR9024NTRPBF" H 7700 3500 50  0001 C CNN "Manufacturer_Part_Number"
-F 6 "942-IRFR9024NTRPBF" H 7700 3500 50  0001 C CNN "Mouser Part Number"
+F 5 "IRLR120NTRPBF" H 7700 3500 50  0001 C CNN "Manufacturer_Part_Number"
+F 6 "942-IRLR120NTRPBF" H 7700 3500 50  0001 C CNN "Mouser Part Number"
 	1    7700 3500
 	1    0    0    -1
@@
 AR Path="/5CB41D9F/E26DE37C" Ref="Q4"  Part="1"
 F 0 "Q4" H 7950 2400 59  0000 L BNN
-F 1 "IRLR120NTRPBF" H 7950 2300 59  0000 L BNN
+F 1 "IRFR9024NTRPBF" H 7950 2300 59  0000 L BNN
 F 2 "Package_TO_SOT_SMD:TO-252-2" H 7700 2400 50  0001 C CNN
 F 3 "https://www.mouser.com/datasheet/2/196/irlr120npbf-1228003.pdf" H 7700 2400 50  0001 C CNN
 F 4 "Infineon" H 7700 2400 50  0001 C CNN "Manufacturer_Name"
-F 5 "IRLR120NTRPBF" H 7700 2400 50  0001 C CNN "Manufacturer_Part_Number"
-F 6 "942-IRLR120NTRPBF" H 7700 2400 50  0001 C CNN "Mouser Part Number"
+F 5 "IRFR9024NTRPBF" H 7700 2400 50  0001 C CNN "Manufacturer_Part_Number"
+F 6 "942-IRFR9024NTRPBF" H 7700 2400 50  0001 C CNN "Mouser Part Number"
 	1    7700 2400
 	1    0    0    -1
@@
 AR Path="/5CB41D9F/4FF9B51F" Ref="Q6"  Part="1"
 F 0 "Q6" H 7950 4500 59  0000 L BNN
-F 1 "IRFR9024NTRPBF" H 7950 4400 59  0000 L BNN
+F 1 "IRLR120NTRPBF" H 7950 4400 59  0000 L BNN
 F 2 "Package_TO_SOT_SMD:TO-252-2" H 7700 4500 50  0001 C CNN
 F 3 "https://www.mouser.com/datasheet/2/196/irfr9024npbf-1228513.pdf" H 7700 4500 50  0001 C CNN
 F 4 "Infineon" H 7700 4500 50  0001 C CNN "Manufacturer_Name"
-F 5 "IRFR9024NTRPBF" H 7700 4500 50  0001 C CNN "Manufacturer_Part_Number"
-F 6 "942-IRFR9024NTRPBF" H 7700 4500 50  0001 C CNN "Mouser Part Number"
+F 5 "IRLR120NTRPBF" H 7700 4500 50  0001 C CNN "Manufacturer_Part_Number"
+F 6 "942-IRLR120NTRPBF" H 7700 4500 50  0001 C CNN "Mouser Part Number"
 	1    7700 4500
 	1    0    0    -1
@@
 AR Path="/5CB41D9F/CE8964FE" Ref="Q8"  Part="1"
 F 0 "Q8" H 7950 6700 59  0000 L BNN
-F 1 "IRFR9024NTRPBF" H 7950 6600 59  0000 L BNN
+F 1 "IRLR120NTRPBF" H 7950 6600 59  0000 L BNN
 F 2 "Package_TO_SOT_SMD:TO-252-2" H 7700 6700 50  0001 C CNN
 F 3 "https://www.mouser.com/datasheet/2/196/irfr9024npbf-1228513.pdf" H 7700 6700 50  0001 C CNN
 F 4 "Infineon" H 7700 6700 50  0001 C CNN "Manufacturer_Name"
-F 5 "IRFR9024NTRPBF" H 7700 6700 50  0001 C CNN "Manufacturer_Part_Number"
-F 6 "942-IRFR9024NTRPBF" H 7700 6700 50  0001 C CNN "Mouser Part Number"
+F 5 "IRLR120NTRPBF" H 7700 6700 50  0001 C CNN "Manufacturer_Part_Number"
+F 6 "942-IRLR120NTRPBF" H 7700 6700 50  0001 C CNN "Mouser Part Number"
 	1    7700 6700
 	1    0    0    -1
@@
 AR Path="/5CB41D9F/EF13FC82" Ref="Q7"  Part="1"
 F 0 "Q7" H 7950 5600 59  0000 L BNN
-F 1 "IRLR120NTRPBF" H 7950 5500 59  0000 L BNN
+F 1 "IRFR9024NTRPBF" H 7950 5500 59  0000 L BNN
 F 2 "Package_TO_SOT_SMD:TO-252-2" H 7700 5600 50  0001 C CNN
 F 3 "https://www.mouser.com/datasheet/2/196/irlr120npbf-1228003.pdf" H 7700 5600 50  0001 C CNN
 F 4 "Infineon" H 7700 5600 50  0001 C CNN "Manufacturer_Name"
-F 5 "IRLR120NTRPBF" H 7700 5600 50  0001 C CNN "Manufacturer_Part_Number"
-F 6 "942-IRLR120NTRPBF" H 7700 5600 50  0001 C CNN "Mouser Part Number"
+F 5 "IRFR9024NTRPBF" H 7700 5600 50  0001 C CNN "Manufacturer_Part_Number"
+F 6 "942-IRFR9024NTRPBF" H 7700 5600 50  0001 C CNN "Mouser Part Number"
 	1    7700 5600
 	1    0    0    -1
